File: untitled.brd (EAGLE design)
At the start: 31 x 16.5 mm, 23 parts, among them IC2 AZ1086, Q1 LMUN2233LT1, Q2 LMUN2233LT1, Q4 12MHz, X1 USB_A_SMT_MALE

Commit message: CH340G rev.2
Parts:
- added CON1: B6B-ZR, jst-zh:B6B-ZR
- J1: device SparkFun-Connectors:1X06_1.27MM -> SparkFun-Connectors:1X01_NO_SILK
- moved J1 24.7 mm to (6.10, 12.4), turned to 0 degrees
- moved C4 15.2 mm to (16.0, 2.41), turned to 270 degrees
- moved C3 15.2 mm to (14.4, 2.41), turned to 270 degrees
- moved Q4 11.4 mm to (12.3, 11.9)
- moved LED2 10.8 mm to (20.3, 3.68)
- moved C2 10.4 mm to (10.7, 11.9), flipped to the top, turned to 270 degrees
- moved R5 9.79 mm to (18.3, 8.64), flipped to the top
- moved Q2 8.90 mm to (22.9, 8.64), turned to 270 degrees
- moved R1 7.89 mm to (22.5, 3.94), flipped to the top, turned to 180 degrees
- moved R4 7.73 mm to (18.3, 5.08), flipped to the top, turned to 90 degrees
- moved Q1 7.67 mm to (23.0, 12.1)
- moved C1 7.29 mm to (14.7, 11.0)
- moved LED3 6.61 mm to (20.3, 9.02)
- moved PTC1 5.80 mm to (5.08, 4.95)
- moved R2 3.84 mm to (22.5, 5.97), flipped to the top, turned to 180 degrees
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Connections:
- net +3V3: now also CON1.2; no longer J1.4
- net +5V: now also J1.1
- net GND: now also CON1.1; no longer J1.6
- net GPIO0: now also CON1.6; no longer J1.5
- net RST: now also CON1.5; no longer J1.1
- net RX: now also CON1.3; no longer J1.3
- net TX: now also CON1.4; no longer J1.2
- net XI: now also Q4.2; no longer Q4.1
- net XO: now also Q4.1; no longer Q4.2
Routing:
- net GND: track 78.8 -> 92.6 mm, vias 3 -> 6
- net RX: track 24.3 -> 12.3 mm, vias 3 -> 0
- net +5V: track 7.03 -> 14.8 mm
- net +3V3: track 41.1 -> 33.9 mm
- net DTR: track 13.8 -> 7.37 mm, vias 0 -> 1
- net N$3: track 7.59 -> 2.12 mm, vias 1 -> 0
- net VUSB: track 6.08 -> 2.09 mm
- net TX: track 20.4 -> 16.7 mm, vias 3 -> 1
- net RST: track 3.04 -> 6.53 mm
- net RTS: track 11.4 -> 8.62 mm, vias 0 -> 1
- net TXD: track 3.00 -> 5.69 mm
- net D-: track 13.8 -> 15.4 mm, vias 0 -> 1
- net XO: track 7.35 -> 8.93 mm
- net N$1: track 6.33 -> 4.92 mm
- net GPIO0: track 5.79 -> 4.67 mm
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Other:
- board size 31 x 16.5 mm -> 31 x 17 mm
- board text added: "5V"
- board text added: "IO0"
- board text added: "Rev.2"
- board text removed: "0"

Commit message: Added.
Parts:
- C3: value 10uF -> 0.1uF
- C4: value 0.1uF -> 10uF
- C5: value 1uF -> 10uF; device generic:SMD1608 -> resistor:C0805
- C6: value 22uF -> 47uF; device generic:SMD1608 -> resistor:C0805
- D1: value RSX101VA-30 -> AVR-M1608C080MTAAB
- LED1, LED2, LED3: device adafruit:CHIPLED_0603 -> adafruit:CHIP-LED0805
- PTC1: device microbuilder:0805 -> microbuilder:1206
- moved C4 6.72 mm to (13.5, 8.64), turned to 90 degrees
- moved C3 2.77 mm to (15.1, 5.08)
- moved C5 1.55 mm to (9.53, 8.76)
- moved R2 1.31 mm to (23.1, 4.83)
- moved R1 1.31 mm to (23.1, 2.79)
- moved C6 1.17 mm to (11.6, 8.76)
- moved R3 1.02 mm to (11.8, 4.57)
- moved LED2 1.02 mm to (20.2, 4.70)
- moved D1 0.80 mm to (7.37, 6.86), turned to 270 degrees
- moved C1 0.63 mm to (14.7, 11.7)
- moved IC2 0.51 mm to (13.0, 5.59)
- moved LED3 0.28 mm to (20.2, 8.76)
- moved Q4 0.25 mm to (12.1, 11.9)
- moved R4 0.25 mm to (18.3, 4.83)
Connections:
- removed net VUSB: D1.+, PTC1.2
- net +5V: now also D1.+, PTC1.2; no longer D1.-
- net GND: now also D1.-
Routing:
- net GND: track 92.6 -> 87.1 mm, vias 6 -> 3
- net RX: track 12.3 -> 9.41 mm
- net VUSB: track 2.09 -> 0.00 mm
- net TX: track 16.7 -> 18.6 mm
- net D+: track 15.3 -> 16.8 mm
- net DTR: track 7.37 -> 8.78 mm
- net TXD: track 5.69 -> 4.53 mm
- net N$2: track 3.71 -> 2.85 mm
- net RXD: track 3.74 -> 4.59 mm
- net D-: track 15.4 -> 16.2 mm
- net +3V3: track 33.9 -> 34.5 mm
- net +5V: track 14.8 -> 15.3 mm
- net XI: track 8.08 -> 8.47 mm, vias 0 -> 1
Other:
- board text added: "3V3"
- board text added: "Rev.3"
- board text removed: "3V"
- board text removed: "Rev.2"
