File: untitled.sch (EAGLE design)
At the start: 23 parts, among them IC2 AZ1086, Q1 LMUN2233LT1, Q2 LMUN2233LT1, Q4 12MHz, X1 USB_A_SMT_MALE

Commit message: CH340G rev.2
Parts:
- added CON1: B6B-ZR, jst-zh:B6B-ZR
- J1: device SparkFun-Connectors:CONN_061.27MM -> SparkFun-Connectors:CONN_01PTH_NO_SILK_YES_STOP
Connections:
- net +3V3: now also CON1.2; no longer J1.4
- net +5V: now also J1.1
- net GND: now also CON1.1; no longer J1.6
- net GPIO0: now also CON1.6; no longer J1.5
- net RST: now also CON1.5; no longer J1.1
- net RX: now also CON1.3; no longer J1.3
- net TX: now also CON1.4; no longer J1.2
- net XI: now also Q4.2; no longer Q4.1
- net XO: now also Q4.1; no longer Q4.2
Other:
- moved on the sheet: Q4
Changed lines of the file:
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@@
 <setting verticaltext="up"/>
 </settings>
-<grid distance="0.1" unitdist="inch" unit="inch" style="lines" multiple="1" display="no" altdistance="0.01" altunitdist="inch" altunit="inch"/>
+<grid distance="0.05" unitdist="inch" unit="inch" style="lines" multiple="1" display="no" altdistance="0.01" altunitdist="inch" altunit="inch"/>
 <layers>
 <layer number="1" name="Top" color="4" fill="1" visible="no" active="no"/>
@@
 <part name="PTC1" library="microbuilder" deviceset="PTC" device="0805"/>
 <part name="X1" library="aitendo" deviceset="USB_A" device="_SMT_MALE"/>
-<part name="J1" library="SparkFun-Connectors" deviceset="CONN_06" device="1.27MM"/>
 <part name="GND6" library="supply" deviceset="GND" device=""/>
 <part name="U$5" library="supply" deviceset="+3V3" device=""/>
@@
 <part name="GND7" library="supply" deviceset="GND" device=""/>
 <part name="U$6" library="supply" deviceset="+3V3" device=""/>
+<part name="U$9" library="supply" deviceset="+5V" device=""/>
+<part name="J1" library="SparkFun-Connectors" deviceset="CONN_01" device="PTH_NO_SILK_YES_STOP"/>
+<part name="CON1" library="jst-zh" deviceset="B6B-ZR" device=""/>
 </parts>
 <sheets>
@@
 <instance part="GND11" gate="1" x="48.26" y="40.64"/>
 <instance part="GND12" gate="1" x="77.47" y="40.64"/>
-<instance part="Q4" gate="G$1" x="83.82" y="27.94"/>
+<instance part="Q4" gate="G$1" x="83.82" y="27.94" rot="R180"/>
 <instance part="R1" gate="G$1" x="115.57" y="30.48"/>
 <instance part="R2" gate="G$1" x="115.57" y="27.94"/>
 <instance part="PTC1" gate="G$1" x="22.86" y="27.94"/>
 <instance part="X1" gate="G$1" x="48.26" y="17.78"/>
-<instance part="J1" gate="G$1" x="137.16" y="71.12" rot="R180"/>
 <instance part="GND6" gate="1" x="121.92" y="58.42"/>
 <instance part="U$5" gate="G$1" x="120.65" y="81.28"/>
@@
 <instance part="GND7" gate="1" x="163.83" y="50.8"/>
 <instance part="U$6" gate="G$1" x="171.45" y="80.01"/>
+<instance part="U$9" gate="G$1" x="30.48" y="76.2"/>
+<instance part="J1" gate="G$1" x="17.78" y="71.12"/>
+<instance part="CON1" gate="G$1" x="151.13" y="63.5" rot="MR180"/>
 </instances>
 <busses>
@@
 <pinref part="C5" gate="G$1" pin="1"/>
 <wire x1="48.26" y1="60.96" x2="48.26" y2="54.61" width="0.1524" layer="91"/>
+</segment>
+<segment>
+<pinref part="U$9" gate="G$1" pin="+5V"/>
+<wire x1="30.48" y1="73.66" x2="30.48" y2="71.12" width="0.1524" layer="91"/>
+<pinref part="J1" gate="G$1" pin="1"/>
+<wire x1="25.4" y1="71.12" x2="30.48" y2="71.12" width="0.1524" layer="91"/>
 </segment>
 </net>
@@
 </segment>
 <segment>
-<pinref part="J1" gate="G$1" pin="6"/>
 <pinref part="GND6" gate="1" pin="GND"/>
-<wire x1="132.08" y1="63.5" x2="121.92" y2="63.5" width="0.1524" layer="91"/>
+<wire x1="146.05" y1="63.5" x2="121.92" y2="63.5" width="0.1524" layer="91"/>
 <wire x1="121.92" y1="63.5" x2="121.92" y2="60.96" width="0.1524" layer="91"/>
 <label x="127" y="63.5" size="1.778" layer="95"/>
+<pinref part="CON1" gate="G$1" pin="1"/>
 </segment>
 <segment>
@@
 <segment>
 <wire x1="72.39" y1="27.94" x2="76.2" y2="27.94" width="0.1524" layer="91"/>
-<wire x1="76.2" y1="27.94" x2="81.28" y2="27.94" width="0.1524" layer="91"/>
 <pinref part="C1" gate="G$1" pin="1"/>
 <wire x1="76.2" y1="27.94" x2="76.2" y2="25.4" width="0.1524" layer="91"/>
 <label x="72.39" y="27.94" size="1.778" layer="95"/>
-<pinref part="Q4" gate="G$1" pin="1"/>
+<pinref part="Q4" gate="G$1" pin="2"/>
+<wire x1="76.2" y1="27.94" x2="81.28" y2="27.94" width="0.1524" layer="91"/>
+<junction x="76.2" y="27.94"/>
 </segment>
 <segment>
@@
 <net name="XO" class="0">
 <segment>
-<wire x1="86.36" y1="27.94" x2="91.44" y2="27.94" width="0.1524" layer="91"/>
 <pinref part="C2" gate="G$1" pin="1"/>
 <wire x1="91.44" y1="27.94" x2="95.25" y2="27.94" width="0.1524" layer="91"/>
 <wire x1="91.44" y1="27.94" x2="91.44" y2="25.4" width="0.1524" layer="91"/>
 <label x="92.71" y="27.94" size="1.778" layer="95"/>
-<pinref part="Q4" gate="G$1" pin="2"/>
+<pinref part="Q4" gate="G$1" pin="1"/>
+<wire x1="91.44" y1="27.94" x2="86.36" y2="27.94" width="0.1524" layer="91"/>
+<junction x="91.44" y="27.94"/>
 </segment>
 <segment>
@@
 </segment>
 <segment>
-<pinref part="J1" gate="G$1" pin="4"/>
-<wire x1="132.08" y1="68.58" x2="120.65" y2="68.58" width="0.1524" layer="91"/>
-<wire x1="120.65" y1="68.58" x2="120.65" y2="78.74" width="0.1524" layer="91"/>
+<wire x1="120.65" y1="66.04" x2="120.65" y2="78.74" width="0.1524" layer="91"/>
 <pinref part="U$5" gate="G$1" pin="+3V3"/>
-<label x="127" y="68.58" size="1.778" layer="95"/>
+<label x="127" y="66.04" size="1.778" layer="95"/>
+<wire x1="120.65" y1="66.04" x2="146.05" y2="66.04" width="0.1524" layer="91"/>
+<pinref part="CON1" gate="G$1" pin="2"/>
 </segment>
 <segment>
@@
 </segment>
 <segment>
-<pinref part="J1" gate="G$1" pin="1"/>
-<wire x1="132.08" y1="76.2" x2="127" y2="76.2" width="0.1524" layer="91"/>
-<label x="127" y="76.2" size="1.778" layer="95"/>
+<wire x1="146.05" y1="73.66" x2="132.08" y2="73.66" width="0.1524" layer="91"/>
+<label x="132.08" y="73.66" size="1.778" layer="95"/>
+<pinref part="CON1" gate="G$1" pin="5"/>
 </segment>
 </net>
@@
 </segment>
 <segment>
-<pinref part="J1" gate="G$1" pin="5"/>
-<wire x1="127" y1="66.04" x2="132.08" y2="66.04" width="0.1524" layer="91"/>
-<label x="127" y="66.04" size="1.778" layer="95"/>
+<wire x1="146.05" y1="76.2" x2="132.08" y2="76.2" width="0.1524" layer="91"/>
+<label x="132.08" y="76.2" size="1.778" layer="95"/>
+<pinref part="CON1" gate="G$1" pin="6"/>
 </segment>
 </net>
@@
 </segment>
 <segment>
-<pinref part="J1" gate="G$1" pin="3"/>
-<wire x1="132.08" y1="71.12" x2="127" y2="71.12" width="0.1524" layer="91"/>
-<label x="127" y="71.12" size="1.778" layer="95"/>
-</segment>
-<segment>
 <pinref part="LED2" gate="G$1" pin="C"/>
 <wire x1="171.45" y1="54.61" x2="171.45" y2="50.8" width="0.1524" layer="91"/>
 <label x="171.45" y="49.53" size="1.778" layer="95"/>
 </segment>
+<segment>
+<wire x1="146.05" y1="68.58" x2="132.08" y2="68.58" width="0.1524" layer="91"/>
+<label x="132.08" y="68.58" size="1.778" layer="95"/>
+<pinref part="CON1" gate="G$1" pin="3"/>
+</segment>
 </net>
 <net name="TX" class="0">
@@
 </segment>
 <segment>
-<pinref part="J1" gate="G$1" pin="2"/>
-<wire x1="132.08" y1="73.66" x2="127" y2="73.66" width="0.1524" layer="91"/>
-<label x="127" y="73.66" size="1.778" layer="95"/>
-</segment>
-<segment>
 <pinref part="LED3" gate="G$1" pin="C"/>
 <wire x1="179.07" y1="54.61" x2="179.07" y2="49.53" width="0.1524" layer="91"/>
 <label x="179.07" y="49.53" size="1.778" layer="95"/>
 </segment>
-</net>
+<segment>
+<wire x1="146.05" y1="71.12" x2="132.08" y2="71.12" width="0.1524" layer="91"/>
+<label x="132.08" y="71.12" size="1.778" layer="95"/>
+<pinref part="CON1" gate="G$1" pin="4"/>
+</segment>
+</net>

Commit message: Added.
Parts:
- C3: value 10uF -> 0.1uF
- C4: value 0.1uF -> 10uF
- C5: value 1uF -> 10uF; device generic:CAPACITOR1608 -> resistor:C-EUC0805
- C6: value 22uF -> 47uF; device generic:CAPACITOR1608 -> resistor:C-EUC0805
- D1: value RSX101VA-30 -> AVR-M1608C080MTAAB
- LED1, LED2, LED3: device adafruit:LEDCHIPLED_0603 -> adafruit:LEDCHIP-LED0805
- PTC1: device microbuilder:PTC0805 -> microbuilder:PTC1206
Connections:
- removed net VUSB: D1.+, PTC1.2
- net +5V: now also D1.+, PTC1.2; no longer D1.-
- net GND: now also D1.-
Other:
- moved on the sheet: C5, C6, D1
Changed lines of the file:
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@@
 <setting verticaltext="up"/>
 </settings>
-<grid distance="0.05" unitdist="inch" unit="inch" style="lines" multiple="1" display="no" altdistance="0.01" altunitdist="inch" altunit="inch"/>
+<grid distance="0.1" unitdist="inch" unit="inch" style="lines" multiple="1" display="no" altdistance="0.01" altunitdist="inch" altunit="inch"/>
 <layers>
 <layer number="1" name="Top" color="4" fill="1" visible="no" active="no"/>
@@
 <part name="Q1" library="for-esp-wroom-02" deviceset="LMUN2233LT1" device=""/>
 <part name="Q2" library="for-esp-wroom-02" deviceset="LMUN2233LT1" device=""/>
-<part name="C3" library="generic" deviceset="CAPACITOR" device="1608" value="10uF"/>
-<part name="C4" library="generic" deviceset="CAPACITOR" device="1608" value="0.1uF"/>
+<part name="C3" library="generic" deviceset="CAPACITOR" device="1608" value="0.1uF"/>
+<part name="C4" library="generic" deviceset="CAPACITOR" device="1608" value="10uF"/>
 <part name="GND2" library="supply" deviceset="GND" device=""/>
 <part name="GND3" library="supply" deviceset="GND" device=""/>
-<part name="D1" library="for-esp32-breakout" deviceset="DIODE*" device="TUMD2" value="RSX101VA-30"/>
+<part name="D1" library="for-esp32-breakout" deviceset="DIODE*" device="TUMD2" value="AVR-M1608C080MTAAB"/>
 <part name="U$3" library="supply" deviceset="+5V" device=""/>
 <part name="GND4" library="supply" deviceset="GND" device=""/>
@@
 <part name="U$4" library="supply" deviceset="+3V3" device=""/>
 <part name="GND10" library="supply" deviceset="GND" device=""/>
-<part name="C5" library="generic" deviceset="CAPACITOR" device="1608" value="1uF"/>
-<part name="C6" library="generic" deviceset="CAPACITOR" device="1608" value="22uF"/>
+<part name="C5" library="resistor" deviceset="C-EU" device="C0805" value="10uF"/>
+<part name="C6" library="resistor" deviceset="C-EU" device="C0805" value="47uF"/>
 <part name="U$7" library="supply" deviceset="+5V" device=""/>
 <part name="U$8" library="supply" deviceset="+3V3" device=""/>
@@
 <part name="R1" library="resistor" deviceset="R-US_" device="R0603" value="470"/>
 <part name="R2" library="resistor" deviceset="R-US_" device="R0603" value="470"/>
-<part name="PTC1" library="microbuilder" deviceset="PTC" device="0805"/>
+<part name="PTC1" library="microbuilder" deviceset="PTC" device="1206"/>
 <part name="X1" library="aitendo" deviceset="USB_A" device="_SMT_MALE"/>
 <part name="GND6" library="supply" deviceset="GND" device=""/>
 <part name="U$5" library="supply" deviceset="+3V3" device=""/>
-<part name="LED1" library="adafruit" deviceset="LED" device="CHIPLED_0603"/>
-<part name="LED2" library="adafruit" deviceset="LED" device="CHIPLED_0603"/>
-<part name="LED3" library="adafruit" deviceset="LED" device="CHIPLED_0603"/>
+<part name="LED1" library="adafruit" deviceset="LED" device="CHIP-LED0805"/>
+<part name="LED2" library="adafruit" deviceset="LED" device="CHIP-LED0805"/>
+<part name="LED3" library="adafruit" deviceset="LED" device="CHIP-LED0805"/>
 <part name="R3" library="resistor" deviceset="R-US_" device="R0603" value="470"/>
 <part name="R4" library="resistor" deviceset="R-US_" device="R0603" value="470"/>
@@
 <part name="J1" library="SparkFun-Connectors" deviceset="CONN_01" device="PTH_NO_SILK_YES_STOP"/>
 <part name="CON1" library="jst-zh" deviceset="B6B-ZR" device=""/>
+<part name="GND8" library="supply" deviceset="GND" device=""/>
 </parts>
 <sheets>
@@
 <instance part="GND2" gate="1" x="167.64" y="12.7"/>
 <instance part="GND3" gate="1" x="175.26" y="12.7"/>
-<instance part="D1" gate="D" x="12.7" y="35.56" rot="R90"/>
+<instance part="D1" gate="D" x="22.86" y="35.56"/>
 <instance part="U$3" gate="G$1" x="12.7" y="45.72"/>
 <instance part="GND4" gate="1" x="12.7" y="5.08"/>
@@
 <instance part="J1" gate="G$1" x="17.78" y="71.12"/>
 <instance part="CON1" gate="G$1" x="151.13" y="63.5" rot="MR180"/>
+<instance part="GND8" gate="1" x="33.02" y="35.56" rot="R90"/>
 </instances>
 <busses>
 </busses>
 <nets>
-<net name="VUSB" class="2">
-<segment>
-<pinref part="D1" gate="D" pin="+"/>
-<wire x1="12.7" y1="27.94" x2="12.7" y2="31.75" width="0.1524" layer="91"/>
-<label x="12.7" y="27.94" size="1.778" layer="95"/>
-<pinref part="PTC1" gate="G$1" pin="2"/>
-<wire x1="17.78" y1="27.94" x2="12.7" y2="27.94" width="0.1524" layer="91"/>
-</segment>
-</net>
 <net name="+5V" class="2">
-<segment>
-<pinref part="U$3" gate="G$1" pin="+5V"/>
-<pinref part="D1" gate="D" pin="-"/>
-<wire x1="12.7" y1="43.18" x2="12.7" y2="39.37" width="0.1524" layer="91"/>
-</segment>
 <segment>
 <pinref part="U$7" gate="G$1" pin="+5V"/>
@@
 <pinref part="J1" gate="G$1" pin="1"/>
 <wire x1="25.4" y1="71.12" x2="30.48" y2="71.12" width="0.1524" layer="91"/>
+</segment>
+<segment>
+<label x="12.7" y="27.94" size="1.778" layer="95"/>
+<pinref part="PTC1" gate="G$1" pin="2"/>
+<wire x1="17.78" y1="27.94" x2="12.7" y2="27.94" width="0.1524" layer="91"/>
+<pinref part="U$3" gate="G$1" pin="+5V"/>
+<wire x1="12.7" y1="43.18" x2="12.7" y2="35.56" width="0.1524" layer="91"/>
+<wire x1="12.7" y1="35.56" x2="12.7" y2="27.94" width="0.1524" layer="91"/>
+<wire x1="12.7" y1="35.56" x2="19.05" y2="35.56" width="0.1524" layer="91"/>
+<junction x="12.7" y="35.56"/>
+<pinref part="D1" gate="D" pin="+"/>
 </segment>
 </net>
@@
 <pinref part="C6" gate="G$1" pin="2"/>
 <pinref part="GND12" gate="1" pin="GND"/>
-<wire x1="77.47" y1="49.53" x2="77.47" y2="43.18" width="0.1524" layer="91"/>
+<wire x1="77.47" y1="46.99" x2="77.47" y2="43.18" width="0.1524" layer="91"/>
 </segment>
 <segment>
 <pinref part="C5" gate="G$1" pin="2"/>
-<wire x1="48.26" y1="49.53" x2="48.26" y2="43.18" width="0.1524" layer="91"/>
+<wire x1="48.26" y1="46.99" x2="48.26" y2="43.18" width="0.1524" layer="91"/>
 <pinref part="GND11" gate="1" pin="GND"/>
 </segment>
@@
 <wire x1="163.83" y1="53.34" x2="163.83" y2="54.61" width="0.1524" layer="91"/>
 </segment>
+<segment>
+<pinref part="D1" gate="D" pin="-"/>
+<pinref part="GND8" gate="1" pin="GND"/>
+<wire x1="26.67" y1="35.56" x2="30.48" y2="35.56" width="0.1524" layer="91"/>
+</segment>
 </net>
